File: Fogger Shield R2 Schematic/Fogger Sheild.sch (EAGLE design)
At the start: 23 parts, among them Q1 MOSFET-NCHANNELFQP30N06L, U1 ARDUINO_SHIELDLABEL

Commit message: Updated Schematic
Parts:
- removed Q1: MOSFET-NCHANNELFQP30N06L, SparkFun-DiscreteSemi:MOSFET-NCHANNELFQP30N06L
- added N-CHMOSFET: V_REG_LD1117VXX, SparkFun-PowerIC:V_REG_LD1117VXX
- U1: value ARDUINO_SHIELDLABEL -> ARDUINO_SHIELDNO_SILK; device SparkFun-Boards:ARDUINO_SHIELDLABEL -> SparkFun-Boards:ARDUINO_SHIELDNO_SILK
Connections:
- net N$25: now also N-CHMOSFET.GND; no longer Q1.S
- net N$26: now also N-CHMOSFET.IN; no longer Q1.D
- net N$27: now also N-CHMOSFET.OUT; no longer Q1.G
Changed lines of the file:
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@@
 </classes>
 <parts>
-<part name="U1" library="SparkFun-Boards" deviceset="ARDUINO_SHIELD" device="LABEL"/>
+<part name="U1" library="SparkFun-Boards" deviceset="ARDUINO_SHIELD" device="NO_SILK" value="ARDUINO_SHIELDNO_SILK"/>
 <part name="R1" library="resistor" deviceset="R-US_" device="0204/5" value="10K"/>
 <part name="R2" library="resistor" deviceset="R-US_" device="0204/2V" value="10K"/>
@@
 <part name="FAN_SPEED_POT" library="SparkFun-Connectors" deviceset="M03" device="PTH" value="1-G 2-+5 3-S"/>
 <part name="D1" library="SparkFun-DiscreteSemi" deviceset="DIODE" device="PTH" value="1N4001"/>
-<part name="Q1" library="SparkFun-DiscreteSemi" deviceset="MOSFET-NCHANNEL" device="FQP30N06L"/>
 <part name="LCD" library="SparkFun-Connectors" deviceset="M04" device="PTH" value="1-G 2-+5 3-SDA 4-SCL"/>
 <part name="FAN" library="SparkFun-Connectors" deviceset="M02" device="PTH"/>
+<part name="N-CHMOSFET" library="SparkFun-PowerIC" deviceset="V_REG_LD1117VXX" device=""/>
 </parts>
 <sheets>
@@
 <instance part="FAN_SPEED_POT" gate="G$1" x="-25.4" y="99.06"/>
 <instance part="D1" gate="G$1" x="78.74" y="-5.08" rot="R180"/>
-<instance part="Q1" gate="G$1" x="93.98" y="5.08"/>
 <instance part="LCD" gate="G$1" x="-22.86" y="53.34" rot="MR180"/>
 <instance part="FAN" gate="G$1" x="78.74" y="-17.78" rot="MR90"/>
+<instance part="N-CHMOSFET" gate="G$1" x="91.44" y="10.16" rot="MR270"/>
 </instances>
 <busses>
@@
 <wire x1="58.42" y1="40.64" x2="101.6" y2="40.64" width="0.2032" layer="91"/>
 <wire x1="101.6" y1="40.64" x2="101.6" y2="22.86" width="0.2032" layer="91"/>
-<wire x1="101.6" y1="22.86" x2="101.6" y2="5.08" width="0.2032" layer="91"/>
+<wire x1="101.6" y1="22.86" x2="101.6" y2="10.16" width="0.2032" layer="91"/>
 <pinref part="R5" gate="G$1" pin="1"/>
 <junction x="101.6" y="22.86"/>
-<wire x1="101.6" y1="5.08" x2="101.6" y2="-2.54" width="0.2032" layer="91"/>
-<wire x1="101.6" y1="-2.54" x2="93.98" y2="-2.54" width="0.2032" layer="91"/>
-<pinref part="Q1" gate="G$1" pin="S"/>
-<wire x1="93.98" y1="-2.54" x2="93.98" y2="0" width="0.2032" layer="91"/>
-<junction x="93.98" y="0"/>
+<pinref part="N-CHMOSFET" gate="G$1" pin="GND"/>
+<wire x1="99.06" y1="10.16" x2="101.6" y2="10.16" width="0.1524" layer="91"/>
+<junction x="99.06" y="10.16"/>
 </segment>
 </net>
@@
 <segment>
 <pinref part="FAN_PWR" gate="G$1" pin="2"/>
-<wire x1="93.98" y1="17.78" x2="81.28" y2="17.78" width="0.2032" layer="91"/>
+<wire x1="93.98" y1="17.78" x2="91.44" y2="17.78" width="0.2032" layer="91"/>
+<wire x1="91.44" y1="17.78" x2="81.28" y2="17.78" width="0.2032" layer="91"/>
 <wire x1="81.28" y1="17.78" x2="81.28" y2="20.32" width="0.2032" layer="91"/>
 <junction x="81.28" y="17.78"/>
-<pinref part="Q1" gate="G$1" pin="D"/>
-<wire x1="93.98" y1="17.78" x2="93.98" y2="10.16" width="0.2032" layer="91"/>
-<junction x="93.98" y="10.16"/>
+<pinref part="N-CHMOSFET" gate="G$1" pin="IN"/>
+<junction x="91.44" y="17.78"/>
 </segment>
 </net>
@@
 <segment>
 <pinref part="FAN" gate="G$1" pin="2"/>
-<wire x1="81.28" y1="5.08" x2="81.28" y2="-2.54" width="0.2032" layer="91"/>
 <pinref part="D1" gate="G$1" pin="A"/>
+<wire x1="81.28" y1="2.54" x2="81.28" y2="-2.54" width="0.2032" layer="91"/>
 <wire x1="81.28" y1="-2.54" x2="81.28" y2="-5.08" width="0.2032" layer="91"/>
 <wire x1="81.28" y1="-5.08" x2="81.28" y2="-7.62" width="0.2032" layer="91"/>
 <junction x="81.28" y="-5.08"/>
 <junction x="81.28" y="-10.16"/>
-<pinref part="Q1" gate="G$1" pin="G"/>
 <wire x1="81.28" y1="-7.62" x2="81.28" y2="-10.16" width="0.2032" layer="91"/>
-<wire x1="86.36" y1="5.08" x2="81.28" y2="5.08" width="0.2032" layer="91"/>
-<junction x="86.36" y="5.08"/>
 <junction x="81.28" y="-7.62"/>
 <junction x="81.28" y="-2.54"/>
-</segment>
-</net>
+<pinref part="N-CHMOSFET" gate="G$1" pin="OUT"/>
+<wire x1="91.44" y1="2.54" x2="81.28" y2="2.54" width="0.1524" layer="91"/>
+<junction x="91.44" y="2.54"/>
+</segment>
+</net>
